Commit message: Correct FANUC browser-ready URDF

File: public/fanuc/urdf/urdf/LRMate-200iD.urdf (robot description, URDF)
Before this commit: robot LRMate-200iD, 7 links, 6 joints
Links:
- removed link base_link
- removed link link_1
- removed link link_2
- removed link link_3
- removed link link_4
- removed link link_5
- removed link link_6
- added link Base; visual mesh filename=package://LRMate-200iD/meshes/base.stl
- added link J1; visual mesh filename=package://LRMate-200iD/meshes/j1.stl
- added link J2; visual mesh filename=package://LRMate-200iD/meshes/j2.stl
- added link J3; visual mesh filename=package://LRMate-200iD/meshes/j3.stl
- added link J4; visual mesh filename=package://LRMate-200iD/meshes/j4.stl
- added link J5; visual mesh filename=package://LRMate-200iD/meshes/j5.stl
- added link J6; visual mesh filename=package://LRMate-200iD/meshes/j6.stl
Joints:
- joint J1: child link_1 -> J1; limit lower=-2.96706 upper=2.96706 effort=100 velocity=2 -> lower=-2.9671 upper=2.9671 effort=0 velocity=0; origin xyz=0 0 0 rpy=0 0 0 -> xyz=0 0 0.042741 rpy=0 0 0; parent base_link -> Base
- joint J2: axis 0 1 0 -> 0 -1 0; child link_2 -> J2; limit lower=-2.13803 upper=2.13803 effort=100 velocity=2 -> lower=-2.1373 upper=2.1373 effort=0 velocity=0; origin xyz=0 0 0.15 rpy=0 0 0 -> xyz=0.05 0 0.28726 rpy=0 0 0; parent link_1 -> J1
- joint J3: axis 0 1 0 -> 0 -1 0; child link_3 -> J3; limit lower=-3.66519 upper=3.66519 effort=100 velocity=2 -> lower=-3.6652 upper=3.6652 effort=0 velocity=0; origin xyz=0 0 0.3 rpy=0 0 0 -> xyz=0 0 0.33 rpy=0 0 0; parent link_2 -> J2
- joint J4: axis 1 0 0 -> -1 0 0; child link_4 -> J4; limit lower=-3.31613 upper=3.31613 effort=100 velocity=2 -> lower=-3.3161 upper=3.3161 effort=0 velocity=0; origin xyz=0 0 0.3 rpy=0 0 0 -> xyz=0.088001 0 0.035027 rpy=0 0 0; parent link_3 -> J3
- joint J5: axis 0 1 0 -> 0 -1 0; child link_5 -> J5; limit lower=-2.18166 upper=2.18166 effort=100 velocity=2 -> lower=-2.1817 upper=2.1817 effort=0 velocity=0; origin xyz=0 0 0.15 rpy=0 0 0 -> xyz=0.2454 0 0 rpy=0 0 0; parent link_4 -> J4
- joint J6: axis 1 0 0 -> -1 0 0; child link_6 -> J6; limit lower=-6.28319 upper=6.28319 effort=100 velocity=2 -> lower=-6.2832 upper=6.2832 effort=0 velocity=0; origin xyz=0 0 0.1 rpy=0 0 0 -> xyz=0.05 0 0 rpy=1.5708 0 0; parent link_5 -> J5
